File: kicad/10-Clock/10-Clock.kicad_sch (KiCad schematic)
At the start: 32 parts, among them SW1 SW_Push, SW2 SW_SPDT, U1 LM555, U2 74LS04, U3 74LS08, U4 LM555, U5 LM555

Commit message: Start emulator and complete clock module
Other:
- note added: "10: Clock"
- title: Clock Module -> 10: Clock Module
Changed lines of the file:
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@@
   (paper "USLetter")
   (title_block
-    (title "Clock Module")
-    (date "2022-01-23")
+    (title "10: Clock Module")
+    (date "2022-02-25")
+    (rev "1.1")
+    (comment 1 "This board is located in Column 1 and in Row 0")
   )
   (junction (at 151.13 81.28) (diameter 0) (color 0 0 0 0)
@@
     (effects (font (size 1.27 1.27)) (justify left bottom))
   )
+  (text "10: Clock" (at 12.7 21.59 0)
+    (effects (font (size 5 5) (thickness 1) bold italic) (justify left bottom))
+  )
   (global_label "HLT" (shape input) (at 87.63 146.05 180) (fields_autoplaced)
